File: Kredsløb print/print v1/_saved_print v1.sch (KiCad schematic (older format))
At the start: 70 parts, among them J1 Conn_01x01_Male, J2 Conn_01x01_Male, J3 Conn_01x01_Male, J4 Conn_01x01_Male, J5 Conn_01x01_Male, Q1 TIP127, Q2 TIP120, Q3 TIP120, Q4 TIP127, Q5 TIP120, U1 esp32, U2 4049

Commit message: schematic and print update
Parts:
- added C? (x2): C, symbol Device:C
- added U?: LM7805_TO220, Package_TO_SOT_THT:TO-220-3_Vertical, symbol Regulator_Linear:LM7805_TO220
Changed lines of the file:
@@
 Wire Wire Line
 	9100 2350 9400 2350
+$Comp
+L Regulator_Linear:LM7805_TO220 U?
+U 1 1 5CA3A1F0
+P 3450 1300
+F 0 "U?" H 3450 1542 50  0000 C CNN
+F 1 "LM7805_TO220" H 3450 1451 50  0000 C CNN
+F 2 "Package_TO_SOT_THT:TO-220-3_Vertical" H 3450 1525 50  0001 C CIN
+F 3 "http://www.fairchildsemi.com/ds/LM/LM7805.pdf" H 3450 1250 50  0001 C CNN
+	1    3450 1300
+	1    0    0    -1
+$EndComp
+$Comp
+L Device:C C?
+U 1 1 5CA3E782
+P 2850 1500
+F 0 "C?" H 2965 1546 50  0000 L CNN
+F 1 "C" H 2965 1455 50  0000 L CNN
+F 2 "" H 2888 1350 50  0001 C CNN
+F 3 "~" H 2850 1500 50  0001 C CNN
+	1    2850 1500
+	1    0    0    -1
+$EndComp
+$Comp
+L Device:C C?
+U 1 1 5CA3FF12
+P 3950 1500
+F 0 "C?" H 4065 1546 50  0000 L CNN
+F 1 "C" H 4065 1455 50  0000 L CNN
+F 2 "" H 3988 1350 50  0001 C CNN
+F 3 "~" H 3950 1500 50  0001 C CNN
+	1    3950 1500
+	1    0    0    -1
+$EndComp
+$Comp
+L power:VCC #PWR?
+U 1 1 5CA41279
+P 1500 900
+F 0 "#PWR?" H 1500 750 50  0001 C CNN
+F 1 "VCC" H 1517 1073 50  0000 C CNN
+F 2 "" H 1500 900 50  0001 C CNN
+F 3 "" H 1500 900 50  0001 C CNN
+	1    1500 900
+	1    0    0    -1
+$EndComp
+$Comp
+L power:VCC #PWR?
+U 1 1 5CA433F6
+P 6550 1000
+F 0 "#PWR?" H 6550 850 50  0001 C CNN
+F 1 "VCC" H 6567 1173 50  0000 C CNN
+F 2 "" H 6550 1000 50  0001 C CNN
+F 3 "" H 6550 1000 50  0001 C CNN
+	1    6550 1000
+	1    0    0    -1
+$EndComp
+$Comp
+L power:VCC #PWR?
+U 1 1 5CA453AB
+P 10100 750
+F 0 "#PWR?" H 10100 600 50  0001 C CNN
+F 1 "VCC" H 10117 923 50  0000 C CNN
+F 2 "" H 10100 750 50  0001 C CNN
+F 3 "" H 10100 750 50  0001 C CNN
+	1    10100 750
+	1    0    0    -1
+$EndComp
+$Comp
+L power:VCC #PWR?
+U 1 1 5CA4674C
+P 10050 3800
+F 0 "#PWR?" H 10050 3650 50  0001 C CNN
+F 1 "VCC" H 10067 3973 50  0000 C CNN
+F 2 "" H 10050 3800 50  0001 C CNN
+F 3 "" H 10050 3800 50  0001 C CNN
+	1    10050 3800
+	1    0    0    -1
+$EndComp
 $EndSCHEMATC

Commit message: faktisk STL
Parts:
- removed J1, J2, J3, J4, J5, J? (x16): Conn_01x01_Male, Connector_PinHeader_1.00mm:PinHeader_1x01_P1.00mm_Vertical, symbol Connector:Conn_01x01_Male
- removed Q1, Q4, Q? (x4): TIP127, Package_TO_SOT_THT:TO-220-3_Vertical, symbol 00-OTG-Transistor:TIP127
- removed Q2, Q3, Q5, Q? (x6): TIP120, TO_SOT_Packages_THT:TO-220_Vertical, symbol 00-OTG-Transistor:TIP120
- removed Q? (x6): BC547, Package_TO_SOT_THT:TO-92_Inline, symbol 00-OTG-Transistor:BC547
- removed R? (x9): R, symbol Device:R
- removed U2: 4049, Package_DIP:DIP-16_W7.62mm_LongPads, symbol 4xxx:4049
- added J? (x26): Conn_01x01_Male, Connector_PinHeader_1.00mm:PinHeader_1x01_P1.00mm_Vertical, symbol Connector:Conn_01x01_Male
- added Q? (x9): TIP120, TO_SOT_Packages_THT:TO-220_Vertical, symbol 00-OTG-Transistor:TIP120
- added Q? (x6): BC547, Package_TO_SOT_THT:TO-92_Inline, symbol 00-OTG-Transistor:BC547
- added Q? (x6): TIP127, Package_TO_SOT_THT:TO-220-3_Vertical, symbol 00-OTG-Transistor:TIP127
- added R? (x9): R, symbol Device:R
- added U? (x3): 4049, Package_DIP:DIP-16_W7.62mm_LongPads, symbol 4xxx:4049
Connections:
- net GND: now also C?.2, C?.2, U?.2 (GND), Q?.3 (E), Q?.3 (E), Q?.3 (E)
- net VCC: now also C?.1, Q?.3 (E), Q?.3 (E), U?.1 (VI), Q?.3 (E), Q?.3 (E), Q?.3 (E), Q?.3 (E), Q?.3 (E), Q?.3 (E)
- net at U1.19 (5V-IN): now also C?.1, U?.3 (VO)
- net at U1.28 (TX2_GIOP17): now also R?.1
- net at U1.29 (VSPI-SS_GIOP5): now also R?.1
- net at U1.30 (VSIP-CLK_GIOP18): now also R?.1
- net at U1.31 (VSPI-MISO_GIOP19): now also R?.1
- net at U1.34 (RX0_GIOP3): now also Q?.2 (B), U?.9
- net at U1.35 (TX0_GIOP1): now also Q?.2 (B), U?.11
- net at U1.36 (I2C-SCL_GIOP22): now also Q?.2 (B), U?.5
- net at U1.37 (VSPI-MOSI_GIOP23): now also Q?.2 (B), U?.3
- net at Q?.1 (B): now also J?.1 (Pin_1); no longer Q?.1 (C)
- net at Q?.2 (B): now also U?.12; no longer U?.2
- net at J?.1 (Pin_1): now also Q?.1 (B)
- new net: J?.1 (Pin_1), Q?.1 (C) (x7)
- new net: Q?.1 (B), R?.2 (x6)
- new net: J?.1 (Pin_1), Q?.2 (C), Q?.2 (C) (x6)
- new net: Q?.2 (C), Q?.3 (E), Q?.3 (E) (x3)
- new net: J?.1 (Pin_1), Q?.1 (B) (x9)
- new net: Q?.2 (B), U?.10
- new net: Q?.3 (E), R?.1 (x6)
- new net: J?.1 (Pin_1), R?.2 (x3)
- new net: Q?.2 (B), U?.4
- new net: Q?.2 (B), U?.2
Other:
- moved on the sheet: C?, U?
