File: Kredsløb print/print v1/arrange test.kicad_pcb (KiCad board)
At the start: 2 copper layers, 77 parts, among them J1 Conn_01x01_Male, J10 Conn_01x01_Male, J11 Conn_01x01_Male, J12 Conn_01x01_Male, J13 Conn_01x01_Male, J14 Conn_01x01_Male, J15 Conn_01x01_Male, J16 Conn_01x01_Male, J17 Conn_01x01_Male, J18 Conn_01x01_Male, J19 Conn_01x01_Male, J2 Conn_01x01_Male, J20 Conn_01x01_Male, J21 Conn_01x01_Male, J22 Conn_01x01_Male, J23 Conn_01x01_Male, J24 Conn_01x01_Male, J25 Conn_01x01_Male, J26 Conn_01x01_Male, J27 Conn_01x01_Male, J28 Conn_01x01_Male, J29 Conn_01x01_Male, J3 Conn_01x01_Male, J30 Conn_01x01_Male, J31 Conn_01x01_Male, J32 Conn_01x01_Male, J4 Conn_01x01_Male, J5 Conn_01x01_Male, J6 Conn_01x01_Male, J7 Conn_01x01_Male, J8 Conn_01x01_Male, J9 Conn_01x01_Male, Q1 BC547, Q10 TIP120, Q11 TIP127, Q12 TIP120, Q13 TIP127, Q14 TIP120, Q15 BC547, Q16 BC547, Q17 BC547, Q18 TIP127, Q19 TIP120, Q2 BC547, Q20 BC547, Q21 TIP127, Q22 TIP120, Q23 TIP120, Q24 TIP120, Q25 TIP127, Q26 TIP120, Q27 TIP127, Q28 TIP120, Q3 BC547, Q4 TIP127, Q5 TIP120, Q6 BC547, Q7 TIP127, Q8 TIP120, Q9 TIP120, U1 esp32, U2 LM7805_TO220, U3 4049

Commit message: kredsløb og ny motor mount
Parts:
- moved U3 53.4 mm to (108.0, 96.5)
- moved C1 32.8 mm to (86.4, 48.3)
- moved C2 15.3 mm to (86.4, 44.5)
- moved U2 15.3 mm to (71.1, 49.5)
Changed lines of the file:
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@@
     (add_net VCC)
   )
+  (module "footprints otg:C_5.00mm" (layer F.Cu)
+    (at 86.36 48.26)
+    (descr "C, Rect series, Radial, pin pitch=2.50mm 5.00mm, , length*width=7*3.5mm^2, Capacitor")
+    (tags "C Rect series Radial pin pitch 2.50mm 5.00mm  length 7mm width 3.5mm Capacitor")
+    (fp_text reference C1 (at 2.54 -2.794) (layer F.SilkS) hide
+      (effects (font (size 1 1) (thickness 0.15)))
+    )
+    (fp_text value C (at 2.54 2.794) (layer F.Fab)
+      (effects (font (size 1 1) (thickness 0.15)))
+    )
+    (fp_text user %R (at 2.54 -2.794) (layer F.Fab) hide
+      (effects (font (size 1 1) (thickness 0.15)))
+    )
+    (fp_line (start 7.52 -2) (end -1.25 -2) (layer F.CrtYd) (width 0.05))
+    (fp_line (start 7.52 2) (end 7.52 -2) (layer F.CrtYd) (width 0.05))
+    (fp_line (start -1.25 2) (end 7.52 2) (layer F.CrtYd) (width 0.05))
+    (fp_line (start -1.25 -2) (end -1.25 2) (layer F.CrtYd) (width 0.05))
+    (fp_line (start 7.39 -1.87) (end 7.39 1.87) (layer F.SilkS) (width 0.12))
+    (fp_line (start -1.12 -1.87) (end -1.12 1.87) (layer F.SilkS) (width 0.12))
+    (fp_line (start -1.12 1.87) (end 7.39 1.87) (layer F.SilkS) (width 0.12))
+    (fp_line (start -1.12 -1.87) (end 7.39 -1.87) (layer F.SilkS) (width 0.12))
+    (fp_line (start 7.27 -1.75) (end -1 -1.75) (layer F.Fab) (width 0.1))
+    (fp_line (start 7.27 1.75) (end 7.27 -1.75) (layer F.Fab) (width 0.1))
+    (fp_line (start -1 1.75) (end 7.27 1.75) (layer F.Fab) (width 0.1))
+    (fp_line (start -1 -1.75) (end -1 1.75) (layer F.Fab) (width 0.1))
+    (pad 2 thru_hole circle (at 6.35 0) (size 1.6 1.6) (drill 0.8) (layers *.Cu *.Mask)
+      (net 2 GND))
+    (pad 1 thru_hole circle (at 0 0) (size 1.6 1.6) (drill 0.8) (layers *.Cu *.Mask)
+      (net 1 "Net-(C1-Pad1)"))
+    (model ${KISYS3DMOD}/Capacitor_THT.3dshapes/C_Rect_L7.0mm_W3.5mm_P2.50mm_P5.00mm.wrl
+      (at (xyz 0 0 0))
+      (scale (xyz 1 1 1))
+      (rotate (xyz 0 0 0))
+    )
+  )
+  (module "footprints otg:C_5.00mm" (layer F.Cu)
+    (at 86.36 44.45)
+    (descr "C, Rect series, Radial, pin pitch=2.50mm 5.00mm, , length*width=7*3.5mm^2, Capacitor")
+    (tags "C Rect series Radial pin pitch 2.50mm 5.00mm  length 7mm width 3.5mm Capacitor")
+    (fp_text reference C2 (at 2.54 -2.794) (layer F.SilkS) hide
+      (effects (font (size 1 1) (thickness 0.15)))
+    )
+    (fp_text value C (at 2.54 2.794) (layer F.Fab)
+      (effects (font (size 1 1) (thickness 0.15)))
+    )
+    (fp_text user %R (at 2.54 -2.794) (layer F.Fab) hide
+      (effects (font (size 1 1) (thickness 0.15)))
+    )
+    (fp_line (start 6.25 -2) (end -1.25 -2) (layer F.CrtYd) (width 0.05))
+    (fp_line (start 6.25 2) (end 6.25 -2) (layer F.CrtYd) (width 0.05))
+    (fp_line (start -1.25 2) (end 6.25 2) (layer F.CrtYd) (width 0.05))
+    (fp_line (start -1.25 -2) (end -1.25 2) (layer F.CrtYd) (width 0.05))
+    (fp_line (start 6.12 -1.87) (end 6.12 1.87) (layer F.SilkS) (width 0.12))
+    (fp_line (start -1.12 -1.87) (end -1.12 1.87) (layer F.SilkS) (width 0.12))
+    (fp_line (start -1.12 1.87) (end 6.12 1.87) (layer F.SilkS) (width 0.12))
+    (fp_line (start -1.12 -1.87) (end 6.12 -1.87) (layer F.SilkS) (width 0.12))
+    (fp_line (start 6 -1.75) (end -1 -1.75) (layer F.Fab) (width 0.1))
+    (fp_line (start 6 1.75) (end 6 -1.75) (layer F.Fab) (width 0.1))
+    (fp_line (start -1 1.75) (end 6 1.75) (layer F.Fab) (width 0.1))
+    (fp_line (start -1 -1.75) (end -1 1.75) (layer F.Fab) (width 0.1))
+    (pad 2 thru_hole circle (at 6.35 0) (size 1.6 1.6) (drill 0.8) (layers *.Cu *.Mask)
+      (net 2 GND))
+    (pad 1 thru_hole circle (at 0 0) (size 1.6 1.6) (drill 0.8) (layers *.Cu *.Mask)
+      (net 3 VCC))
+    (pad 2 thru_hole circle (at 3.75 0) (size 1.6 1.6) (drill 0.8) (layers *.Cu *.Mask)
+      (net 2 GND))
+    (pad 1 thru_hole circle (at 1.25 0) (size 1.6 1.6) (drill 0.8) (layers *.Cu *.Mask)
+      (net 3 VCC))
+    (model ${KISYS3DMOD}/Capacitor_THT.3dshapes/C_Rect_L7.0mm_W3.5mm_P2.50mm_P5.00mm.wrl
+      (at (xyz 0 0 0))
+      (scale (xyz 1 1 1))
+      (rotate (xyz 0 0 0))
+    )
+  )
   (module Package_DIP:DIP-16_W7.62mm_LongPads (layer F.Cu)
-    (at 124.46 147.32)
+    (at 107.95 96.52)
     (descr "16-lead though-hole mounted DIP package, row spacing 7.62 mm (300 mils), LongPads")
     (tags "THT DIP DIL PDIP 2.54mm 7.62mm 300mil LongPads")
@@
   )
   (module Package_TO_SOT_THT:TO-220-3_Vertical (layer F.Cu)
-    (at 72.39 34.29)
+    (at 71.12 49.53)
     (descr "TO-220-3, Vertical, RM 2.54mm, see https://www.vishay.com/docs/66542/to-220-1.pdf")
     (tags "TO-220-3 Vertical RM 2.54mm")
@@
       (at (xyz 0 0 0))
       (scale (xyz 1 1 1))
-      (rotate (xyz 0 0 0))
-    )
-  )
-  (module "footprints otg:C_5.00mm" (layer F.Cu)
-    (at 87.63 29.21)
-    (descr "C, Rect series, Radial, pin pitch=2.50mm 5.00mm, , length*width=7*3.5mm^2, Capacitor")
-    (tags "C Rect series Radial pin pitch 2.50mm 5.00mm  length 7mm width 3.5mm Capacitor")
-    (fp_text reference C2 (at 2.54 -2.794) (layer F.SilkS) hide
-      (effects (font (size 1 1) (thickness 0.15)))
-    )
-    (fp_text value C (at 2.54 2.794) (layer F.Fab)
-      (effects (font (size 1 1) (thickness 0.15)))
-    )
-    (fp_text user %R (at 2.54 -2.794) (layer F.Fab) hide
-      (effects (font (size 1 1) (thickness 0.15)))
-    )
-    (fp_line (start 6.25 -2) (end -1.25 -2) (layer F.CrtYd) (width 0.05))
-    (fp_line (start 6.25 2) (end 6.25 -2) (layer F.CrtYd) (width 0.05))
-    (fp_line (start -1.25 2) (end 6.25 2) (layer F.CrtYd) (width 0.05))
-    (fp_line (start -1.25 -2) (end -1.25 2) (layer F.CrtYd) (width 0.05))
-    (fp_line (start 6.12 -1.87) (end 6.12 1.87) (layer F.SilkS) (width 0.12))
-    (fp_line (start -1.12 -1.87) (end -1.12 1.87) (layer F.SilkS) (width 0.12))
-    (fp_line (start -1.12 1.87) (end 6.12 1.87) (layer F.SilkS) (width 0.12))
-    (fp_line (start -1.12 -1.87) (end 6.12 -1.87) (layer F.SilkS) (width 0.12))
-    (fp_line (start 6 -1.75) (end -1 -1.75) (layer F.Fab) (width 0.1))
-    (fp_line (start 6 1.75) (end 6 -1.75) (layer F.Fab) (width 0.1))
-    (fp_line (start -1 1.75) (end 6 1.75) (layer F.Fab) (width 0.1))
-    (fp_line (start -1 -1.75) (end -1 1.75) (layer F.Fab) (width 0.1))
-    (pad 2 thru_hole circle (at 5 0) (size 1.6 1.6) (drill 0.8) (layers *.Cu *.Mask)
-      (net 2 GND))
-    (pad 1 thru_hole circle (at 0 0) (size 1.6 1.6) (drill 0.8) (layers *.Cu *.Mask)
-      (net 3 VCC))
-    (pad 2 thru_hole circle (at 3.75 0) (size 1.6 1.6) (drill 0.8) (layers *.Cu *.Mask)
-      (net 2 GND))
-    (pad 1 thru_hole circle (at 1.25 0) (size 1.6 1.6) (drill 0.8) (layers *.Cu *.Mask)
-      (net 3 VCC))
-    (model ${KISYS3DMOD}/Capacitor_THT.3dshapes/C_Rect_L7.0mm_W3.5mm_P2.50mm_P5.00mm.wrl
-      (at (xyz 0 0 0))
-      (scale (xyz 1 1 1))
-      (rotate (xyz 0 0 0))
-    )
-  )
-  (module "footprints otg:C_5.00mm" (layer F.Cu)
-    (at 59.69 29.21)
-    (descr "C, Rect series, Radial, pin pitch=2.50mm 5.00mm, , length*width=7*3.5mm^2, Capacitor")
-    (tags "C Rect series Radial pin pitch 2.50mm 5.00mm  length 7mm width 3.5mm Capacitor")
-    (fp_text reference C1 (at 2.54 -2.794) (layer F.SilkS) hide
-      (effects (font (size 1 1) (thickness 0.15)))
-    )
-    (fp_text value C (at 2.54 2.794) (layer F.Fab)
-      (effects (font (size 1 1) (thickness 0.15)))
-    )
-    (fp_text user %R (at 2.54 -2.794) (layer F.Fab) hide
-      (effects (font (size 1 1) (thickness 0.15)))
-    )
-    (fp_line (start 6.25 -2) (end -1.25 -2) (layer F.CrtYd) (width 0.05))
-    (fp_line (start 6.25 2) (end 6.25 -2) (layer F.CrtYd) (width 0.05))
-    (fp_line (start -1.25 2) (end 6.25 2) (layer F.CrtYd) (width 0.05))
-    (fp_line (start -1.25 -2) (end -1.25 2) (layer F.CrtYd) (width 0.05))
-    (fp_line (start 6.12 -1.87) (end 6.12 1.87) (layer F.SilkS) (width 0.12))
-    (fp_line (start -1.12 -1.87) (end -1.12 1.87) (layer F.SilkS) (width 0.12))
-    (fp_line (start -1.12 1.87) (end 6.12 1.87) (layer F.SilkS) (width 0.12))
-    (fp_line (start -1.12 -1.87) (end 6.12 -1.87) (layer F.SilkS) (width 0.12))
-    (fp_line (start 6 -1.75) (end -1 -1.75) (layer F.Fab) (width 0.1))
-    (fp_line (start 6 1.75) (end 6 -1.75) (layer F.Fab) (width 0.1))
-    (fp_line (start -1 1.75) (end 6 1.75) (layer F.Fab) (width 0.1))
-    (fp_line (start -1 -1.75) (end -1 1.75) (layer F.Fab) (width 0.1))
-    (pad 2 thru_hole circle (at 5 0) (size 1.6 1.6) (drill 0.8) (layers *.Cu *.Mask)
-      (net 2 GND))
-    (pad 1 thru_hole circle (at 0 0) (size 1.6 1.6) (drill 0.8) (layers *.Cu *.Mask)
-      (net 1 "Net-(C1-Pad1)"))
-    (pad 2 thru_hole circle (at 3.75 0) (size 1.6 1.6) (drill 0.8) (layers *.Cu *.Mask)
-      (net 2 GND))
-    (pad 1 thru_hole circle (at 1.25 0) (size 1.6 1.6) (drill 0.8) (layers *.Cu *.Mask)
-      (net 1 "Net-(C1-Pad1)"))
-    (model ${KISYS3DMOD}/Capacitor_THT.3dshapes/C_Rect_L7.0mm_W3.5mm_P2.50mm_P5.00mm.wrl
-      (at (xyz 0 0 0))
-      (scale (xyz 1 1 1))
