File: Kredsløb print/print v1/print v1.kicad_pcb (KiCad board)
At the start: 2 copper layers, 53 parts, among them J1 Conn_01x01_Male, J10 Conn_01x01_Male, J11 Conn_01x01_Male, J12 Conn_01x01_Male, J13 Conn_01x01_Male, J14 Conn_01x01_Male, J15 Conn_01x01_Male, J16 Conn_01x01_Male, J17 Conn_01x01_Male, J18 Conn_01x01_Male, J19 Conn_01x01_Male, J2 Conn_01x01_Male, J20 Conn_01x01_Male, J21 Conn_01x01_Male, J22 Conn_01x01_Male, J23 Conn_01x01_Male, J24 Conn_01x01_Male, J25 Conn_01x01_Male, J26 Conn_01x01_Male, J27 Conn_01x01_Male, J28 Conn_01x01_Male, J29 Conn_01x01_Male, J3 Conn_01x01_Male, J30 Conn_01x01_Male, J31 Conn_01x01_Male, J32 Conn_01x01_Male, J4 Conn_01x01_Male, J5 Conn_01x01_Male, J6 Conn_01x01_Male, J7 Conn_01x01_Male, J8 Conn_01x01_Male, J9 Conn_01x01_Male, Q1 BC547, Q11 TIP127, Q13 TIP127, Q15 BC547, Q16 BC547, Q17 BC547, Q18 TIP127, Q2 BC547, Q20 BC547, Q21 TIP127, Q25 TIP127, Q27 TIP127, Q3 BC547, Q4 TIP127, Q6 BC547, Q7 TIP127, U1 esp32, U2 LM7805_TO220, U3 4049

Commit message: kredsløb og ny motor mount
Parts:
- added Q10: TIP120, Package_TO_SOT_THT:TO-220-3_Vertical, F.Cu at (162.6, 83.8)
- added Q12: TIP120, Package_TO_SOT_THT:TO-220-3_Vertical, F.Cu at (168.9, 148.6)
- added Q14: TIP120, Package_TO_SOT_THT:TO-220-3_Vertical, F.Cu at (177.8, 61.0)
- added Q19: TIP120, Package_TO_SOT_THT:TO-220-3_Vertical, F.Cu at (217.2, 128.3)
- added Q22: TIP120, Package_TO_SOT_THT:TO-220-3_Vertical, F.Cu at (227.3, 55.9)
- added Q23: TIP120, Package_TO_SOT_THT:TO-220-3_Vertical, F.Cu at (227.3, 151.1)
- added Q24: TIP120, Package_TO_SOT_THT:TO-220-3_Vertical, F.Cu at (237.5, 78.7)
- added Q26: TIP120, Package_TO_SOT_THT:TO-220-3_Vertical, F.Cu at (242.6, 128.3)
- added Q28: TIP120, Package_TO_SOT_THT:TO-220-3_Vertical, F.Cu at (252.7, 55.9)
- added Q5: TIP120, Package_TO_SOT_THT:TO-220-3_Vertical, F.Cu at (143.5, 148.6)
- added Q8: TIP120, Package_TO_SOT_THT:TO-220-3_Vertical, F.Cu at (152.4, 61.0)
- added Q9: TIP120, Package_TO_SOT_THT:TO-220-3_Vertical, F.Cu at (153.7, 171.4)
- added R1: R, footprints otg:R_vandret, F.Cu at (133.3, 142.2)
- added R10: R, footprints otg:R_vandret, F.Cu at (218.4, 151.1)
- added R11: R, footprints otg:R_vandret, F.Cu at (228.6, 68.6)
- added R12: R, footprints otg:R_vandret, F.Cu at (228.6, 78.7)
- added R2: R, footprints otg:R_vandret, F.Cu at (142.2, 50.8)
- added R3: R, footprints otg:R_vandret, F.Cu at (144.8, 161.3)
- added R4: R, footprints otg:R_vandret, F.Cu at (144.8, 171.4)
- added R5: R, footprints otg:R_vandret, F.Cu at (149.9, 74.9)
- added R6: R, footprints otg:R_vandret, F.Cu at (147.3, 83.8)
- added R7: R, footprints otg:R_vandret, F.Cu at (207.0, 121.9)
- added R8: R, footprints otg:R_vandret, F.Cu at (217.2, 49.5)
- added R9: R, footprints otg:R_vandret, F.Cu at (218.4, 141.0)
- C1, C2: footprint footprints otg:C_5.00mm -> Custom footprints:C_6.00mm
- moved Q27 169.2 mm to (252.7, 36.8)
- moved C2 155.4 mm to (69.8, 24.1)
- moved J27 147.7 mm to (237.5, 26.7)
- moved J31 145.9 mm to (242.6, 26.7)
- moved Q25 145.6 mm to (242.6, 109.2)
- moved C1 137.9 mm to (91.4, 22.9), turned to 180 degrees
- moved J21 135.5 mm to (227.3, 99.1)
- moved J30 121.9 mm to (241.3, 47.0)
- moved J11 120.0 mm to (162.6, 31.8)
- moved J20 118.4 mm to (222.2, 58.4)
- moved J23 116.3 mm to (227.3, 141.0)
- moved U2 115.9 mm to (72.4, 34.3)
- moved J32 115.5 mm to (242.6, 68.6)
- moved J15 114.5 mm to (167.6, 31.8)
- moved U3 101.5 mm to (62.2, 44.5)
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