File: Kredsløb print/Prints V2/Print V2/Print V2.kicad_pcb (KiCad board)
At the start: 2 copper layers, 77 parts, among them J1 Conn_01x01_Male, J10 Conn_01x01_Male, J11 Conn_01x01_Male, J12 Conn_01x01_Male, J13 Conn_01x01_Male, J14 Conn_01x01_Male, J15 Conn_01x01_Male, J16 Conn_01x01_Male, J17 Conn_01x01_Male, J18 Conn_01x01_Male, J19 Conn_01x01_Male, J2 Conn_01x01_Male, J20 Conn_01x01_Male, J21 Conn_01x01_Male, J22 Conn_01x01_Male, J23 Conn_01x01_Male, J24 Conn_01x01_Male, J25 Conn_01x01_Male, J26 Conn_01x01_Male, J27 Conn_01x01_Male, J28 Conn_01x01_Male, J29 Conn_01x01_Male, J3 Conn_01x01_Male, J30 Conn_01x01_Male, J31 Conn_01x01_Male, J32 Conn_01x01_Male, J4 Conn_01x01_Male, J5 Conn_01x01_Male, J6 Conn_01x01_Male, J7 Conn_01x01_Male, J8 Conn_01x01_Male, J9 Conn_01x01_Male, Q1 BC547, Q10 TIP120, Q11 TIP127, Q12 TIP120, Q13 TIP127, Q14 TIP120, Q15 BC547, Q16 BC547, Q17 BC547, Q18 TIP127, Q19 TIP120, Q2 BC547, Q20 BC547, Q21 TIP127, Q22 TIP120, Q23 TIP120, Q24 TIP120, Q25 TIP127, Q26 TIP120, Q27 TIP127, Q28 TIP120, Q3 BC547, Q4 TIP127, Q5 TIP120, Q6 BC547, Q7 TIP127, Q8 TIP120, Q9 TIP120, U1 esp32, U2 LM7805_TO220, U3 4049

Commit message: kredsløb og ny motor mount
Parts:
- C1, C2: footprint footprints otg:C_5.00mm -> Custom footprints:C_6.00mm
- U1: value esp32 -> LM7805_TO220; footprint footprints otg:ESP32_mcu -> Package_TO_SOT_THT:TO-220-3_Vertical
- U2: value LM7805_TO220 -> esp32; footprint Package_TO_SOT_THT:TO-220-3_Vertical -> footprints otg:ESP32_mcu
- moved C2 119.9 mm to (55.9, 144.8), turned to 90 degrees
- moved C1 117.1 mm to (40.6, 144.8), turned to 90 degrees
- moved U3 103.6 mm to (38.1, 90.2), turned to 90 degrees
- moved U2 85.9 mm to (61.0, 119.4)
- moved U1 54.1 mm to (45.7, 144.8)
Connections:
- C1 pad 1: Net-(C1-Pad1) -> VCC
- C2 pad 1: VCC -> Net-(C2-Pad1)
- U1 pad 1: Net-(U1-Pad1) -> VCC
- U1 pad 2: Net-(U1-Pad2) -> GND
- U1 pad 3: Net-(U1-Pad3) -> Net-(C2-Pad1)
- U2 pad 1: VCC -> Net-(U2-Pad1)
- U2 pad 2: GND -> Net-(U2-Pad2)
- U2 pad 3: Net-(C1-Pad1) -> Net-(U2-Pad3)

Commit message: Lotsa stuff
Parts:
- added J33: Conn_01x01, Custom footprints:Power_wire_pad, F.Cu at (29.2, 116.8)
- added J34: Conn_01x01, Custom footprints:Power_wire_pad, F.Cu at (29.2, 122.8)
Connections:
- U2 pad 34: Net-(Q3-Pad2) -> Net-(Q17-Pad2)
- U2 pad 35: Net-(Q17-Pad2) -> Net-(Q3-Pad2)
Changed lines of the file:
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@@
     (tracks 0)
     (zones 0)
-    (modules 77)
+    (modules 79)
     (nets 96)
   )
@@
     (solder_mask_min_width 0.25)
     (aux_axis_origin 0 0)
-    (visible_elements FFFFFF7F)
+    (visible_elements 7FFFFFFF)
     (pcbplotparams
       (layerselection 0x010fc_ffffffff)
@@
     (add_net VCC)
   )
+  (module "Custom footprints:Power_wire_pad" (layer F.Cu)
+    (at 29.21 122.85 270)
+    (descr "C, Rect series, Radial, pin pitch=2.50mm 5.00mm, , length*width=7*3.5mm^2, Capacitor")
+    (tags "C Rect series Radial pin pitch 2.50mm 5.00mm  length 7mm width 3.5mm Capacitor")
+    (fp_text reference J34 (at 2.54 -2.794 270) (layer F.SilkS) hide
+      (effects (font (size 1 1) (thickness 0.15)))
+    )
+    (fp_text value Conn_01x01 (at 2.54 2.794 270) (layer F.Fab)
+      (effects (font (size 1 1) (thickness 0.15)))
+    )
+    (fp_text user %R (at 2.54 -2.794 270) (layer F.Fab) hide
+      (effects (font (size 1 1) (thickness 0.15)))
+    )
+    (fp_line (start 2.44 -2) (end -2.52 -2) (layer F.CrtYd) (width 0.05))
+    (fp_line (start 2.44 2) (end 2.44 -2) (layer F.CrtYd) (width 0.05))
+    (fp_line (start -2.52 2) (end 2.44 2) (layer F.CrtYd) (width 0.05))
+    (fp_line (start -2.52 -2) (end -2.52 2) (layer F.CrtYd) (width 0.05))
+    (fp_line (start 2.31 -1.87) (end 2.31 1.87) (layer F.SilkS) (width 0.12))
+    (fp_line (start -2.39 -1.87) (end -2.39 1.87) (layer F.SilkS) (width 0.12))
+    (fp_line (start -2.39 1.87) (end 2.31 1.87) (layer F.SilkS) (width 0.12))
+    (fp_line (start -2.39 -1.87) (end 2.31 -1.87) (layer F.SilkS) (width 0.12))
+    (fp_line (start 2.19 -1.75) (end -2.27 -1.75) (layer F.Fab) (width 0.1))
+    (fp_line (start 2.19 1.75) (end 2.19 -1.75) (layer F.Fab) (width 0.1))
+    (fp_line (start -2.27 1.75) (end 2.19 1.75) (layer F.Fab) (width 0.1))
+    (fp_line (start -2.27 -1.75) (end -2.27 1.75) (layer F.Fab) (width 0.1))
+    (pad 1 smd roundrect (at 0 0 270) (size 3.5 3) (layers F.Cu F.Paste F.Mask) (roundrect_rratio 0.25)
+      (net 2 VCC))
+    (model ${KISYS3DMOD}/Capacitor_THT.3dshapes/C_Rect_L7.0mm_W3.5mm_P2.50mm_P5.00mm.wrl
+      (at (xyz 0 0 0))
+      (scale (xyz 1 1 1))
+      (rotate (xyz 0 0 0))
+    )
+  )
+  (module "Custom footprints:Power_wire_pad" (layer F.Cu)
+    (at 29.21 116.84 270)
+    (descr "C, Rect series, Radial, pin pitch=2.50mm 5.00mm, , length*width=7*3.5mm^2, Capacitor")
+    (tags "C Rect series Radial pin pitch 2.50mm 5.00mm  length 7mm width 3.5mm Capacitor")
+    (fp_text reference J33 (at 2.54 -2.794 270) (layer F.SilkS) hide
+      (effects (font (size 1 1) (thickness 0.15)))
+    )
+    (fp_text value Conn_01x01 (at 2.54 2.794 270) (layer F.Fab)
+      (effects (font (size 1 1) (thickness 0.15)))
+    )
+    (fp_text user %R (at 2.54 -2.794 270) (layer F.Fab) hide
+      (effects (font (size 1 1) (thickness 0.15)))
+    )
+    (fp_line (start 2.44 -2) (end -2.52 -2) (layer F.CrtYd) (width 0.05))
+    (fp_line (start 2.44 2) (end 2.44 -2) (layer F.CrtYd) (width 0.05))
+    (fp_line (start -2.52 2) (end 2.44 2) (layer F.CrtYd) (width 0.05))
+    (fp_line (start -2.52 -2) (end -2.52 2) (layer F.CrtYd) (width 0.05))
+    (fp_line (start 2.31 -1.87) (end 2.31 1.87) (layer F.SilkS) (width 0.12))
+    (fp_line (start -2.39 -1.87) (end -2.39 1.87) (layer F.SilkS) (width 0.12))
+    (fp_line (start -2.39 1.87) (end 2.31 1.87) (layer F.SilkS) (width 0.12))
+    (fp_line (start -2.39 -1.87) (end 2.31 -1.87) (layer F.SilkS) (width 0.12))
+    (fp_line (start 2.19 -1.75) (end -2.27 -1.75) (layer F.Fab) (width 0.1))
+    (fp_line (start 2.19 1.75) (end 2.19 -1.75) (layer F.Fab) (width 0.1))
+    (fp_line (start -2.27 1.75) (end 2.19 1.75) (layer F.Fab) (width 0.1))
+    (fp_line (start -2.27 -1.75) (end -2.27 1.75) (layer F.Fab) (width 0.1))
+    (pad 1 smd roundrect (at 0 0 270) (size 3.5 3) (layers F.Cu F.Paste F.Mask) (roundrect_rratio 0.25)
+      (net 1 GND))
+    (model ${KISYS3DMOD}/Capacitor_THT.3dshapes/C_Rect_L7.0mm_W3.5mm_P2.50mm_P5.00mm.wrl
+      (at (xyz 0 0 0))
+      (scale (xyz 1 1 1))
+      (rotate (xyz 0 0 0))
+    )
+  )
   (module Package_DIP:DIP-16_W7.62mm_LongPads (layer F.Cu)
     (at 38.1 90.17 90)
@@
       (net 51 "Net-(Q15-Pad2)"))
     (pad 35 thru_hole oval (at -12.7 -12.7 90) (size 4.4 2) (drill 0.762) (layers *.Cu *.Mask)
+      (net 41 "Net-(Q3-Pad2)"))
+    (pad 34 thru_hole oval (at -10.16 -12.7 90) (size 4.4 2) (drill 0.762) (layers *.Cu *.Mask)
       (net 55 "Net-(Q17-Pad2)"))
-    (pad 34 thru_hole oval (at -10.16 -12.7 90) (size 4.4 2) (drill 0.762) (layers *.Cu *.Mask)
-      (net 41 "Net-(Q3-Pad2)"))
     (pad 33 thru_hole oval (at -7.62 -12.7 90) (size 4.4 2) (drill 0.762) (layers *.Cu *.Mask)
       (net 68 "Net-(U2-Pad33)"))

Commit message: stuff
Parts:
- moved C1 61.3 mm to (26.7, 85.1), turned to 0 degrees
- moved U1 57.8 mm to (26.7, 90.2), turned to 270 degrees
- moved C2 53.2 mm to (26.7, 100.3), turned to 0 degrees
- moved U3 1.27 mm to (38.1, 91.4)
Connections:
- U3 pad 1: (no net) -> Net-(C2-Pad1)
- U3 pad 8: (no net) -> GND
