File: Kredsløb print/Prints V2/Print V2/Print V2_ESP-signalsystem og strøm routing.kicad_pcb (KiCad board)
At the start: 2 copper layers, 24 parts, among them J1 Conn_01x01, J17 Conn_01x01, J18 Conn_01x01, J19 Conn_01x01, J2 Conn_01x01, J20 Conn_01x01, J21 Conn_01x02, J22 Conn_01x02, J23 Conn_01x02, J24 Conn_01x02, J3 Conn_01x01, J33 Conn_01x01, J34 Conn_01x01, J4 Conn_01x01, J5 Conn_01x01, J6 Conn_01x01, J7 Conn_01x01, J8 Conn_01x01, J9 Conn_01x19, U1 LM7805_TO220, U2 esp32, U3 4049

Commit message: Stuff
Parts:
- J1, J17, J18, J19, J2, J20, J3, J4, J5, J6, J7, J8: footprint Connector_PinHeader_2.54mm:PinHeader_1x01_P2.54mm_Vertical -> Connector_PinSocket_2.54mm:PinSocket_1x01_P2.54mm_Vertical
- J21, J22, J23, J24: footprint Connector_PinHeader_2.54mm:PinHeader_1x02_P2.54mm_Vertical -> Connector_PinSocket_2.54mm:PinSocket_1x02_P2.54mm_Vertical
- J9: footprint Connector_PinHeader_2.54mm:PinHeader_1x19_P2.54mm_Vertical -> Connector_PinSocket_2.54mm:PinSocket_1x19_P2.54mm_Vertical
