File: Kredsløb print/Prints V2/Print V2/Print V2_H-bro og PWM input.kicad_pcb (KiCad board)
At the start: 2 copper layers, 19 parts, among them J1 Conn_01x01_Male, J19 Conn_01x01_Male, J2 Conn_01x01_Male, J20 Conn_01x01_Male, J28 Conn_01x01_Male, J3 Conn_01x01_Male, J30 Conn_01x01_Male, J4 Conn_01x01_Male, J5 Conn_01x01_Male, Q17 BC547, Q20 BC547, Q21 TIP127, Q22 TIP120, Q24 TIP120, Q27 TIP127, Q28 TIP120

Commit message: idk
Changed lines of the file:
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@@
     (0 F.Cu signal)
     (31 B.Cu signal)
-    (32 B.Adhes user hide)
-    (33 F.Adhes user hide)
-    (34 B.Paste user hide)
-    (35 F.Paste user hide)
-    (36 B.SilkS user hide)
-    (37 F.SilkS user hide)
-    (38 B.Mask user hide)
-    (39 F.Mask user hide)
+    (32 B.Adhes user)
+    (33 F.Adhes user)
+    (34 B.Paste user)
+    (35 F.Paste user)
+    (36 B.SilkS user)
+    (37 F.SilkS user)
+    (38 B.Mask user)
+    (39 F.Mask user)
     (40 Dwgs.User user hide)
-    (41 Cmts.User user hide)
-    (42 Eco1.User user hide)
-    (43 Eco2.User user hide)
-    (44 Edge.Cuts user hide)
-    (45 Margin user hide)
+    (41 Cmts.User user)
+    (42 Eco1.User user)
+    (43 Eco2.User user)
+    (44 Edge.Cuts user)
+    (45 Margin user)
     (46 B.CrtYd user hide)
     (47 F.CrtYd user hide)
-    (48 B.Fab user hide)
+    (48 B.Fab user)
     (49 F.Fab user hide)
   )
@@
     (descr "TO-92 leads in-line, narrow, oval pads, drill 0.75mm (see NXP sot054_po.pdf)")
     (tags "to-92 sc-43 sc-43a sot54 PA33 transistor")
-    (fp_text reference Q20 (at 1.27 -3.56 270) (layer F.SilkS)
+    (fp_text reference Q20 (at 1.27 2.54 270) (layer F.SilkS)
       (effects (font (size 1 1) (thickness 0.15)))
     )
@@
     (connect_pads (clearance 0.508))
     (min_thickness 0.254)
-    (fill yes (arc_segments 32) (thermal_gap 0.508) (thermal_bridge_width 0.508))
+    (fill (arc_segments 32) (thermal_gap 0.508) (thermal_bridge_width 0.508))
     (polygon
       (pts

Commit message: Stuff
Parts:
- removed J19, J20, J28, J30: Conn_01x01_Male, Connector_PinHeader_2.54mm:PinHeader_1x01_P2.54mm_Vertical
- added J6: Conn_01x01, Custom footprints:Wire_hole, F.Cu at (144.8, 67.3)
- added J7: Conn_01x01, Custom footprints:Wire_hole, F.Cu at (151.8, 94.0)
- added J8: Conn_01x02, Connector_PinSocket_2.54mm:PinSocket_1x02_P2.54mm_Vertical, F.Cu at (146.1, 79.4)
- J1, J2, J3, J4, J5: value Conn_01x01_Male -> Conn_01x01; footprint Connector_PinHeader_2.54mm:PinHeader_1x01_P2.54mm_Vertical -> Custom footprints:Wire_hole
- moved J5 31.2 mm to (125.7, 79.4)
- moved J4 17.1 mm to (127.6, 69.8)
- moved J3 14.0 mm to (142.2, 79.4)
- moved J2 2.54 mm to (128.3, 83.8)
- moved J1 2.54 mm to (127.6, 66.0)
Connections:
- J5 pad 1: GND -> Net-(J5-Pad1)
- Q20 pad 1: Net-(J19-Pad1) -> Net-(J4-Pad1)
- Q20 pad 2: Net-(J3-Pad1) -> Net-(J5-Pad1)
- Q21 pad 1: Net-(J20-Pad1) -> Net-(J3-Pad1)
- Q21 pad 3: Net-(J4-Pad1) -> Net-(J6-Pad1)
- Q27 pad 3: Net-(J4-Pad1) -> Net-(J6-Pad1)
Routing:
- net Net-(J6-Pad1): track 0.00 -> 12.1 mm
- net Net-(J19-Pad1): track 8.16 -> 0.00 mm
- net Net-(J4-Pad1): track 12.1 -> 8.16 mm
- net Net-(J5-Pad1): track 0.00 -> 3.81 mm
- net Net-(J20-Pad1): track 3.81 -> 0.00 mm
